Commit message: Add friction to wheels

File: omnibot_description/urdf/omnibot_gazebo.xacro (robot description, xacro)
@@ -1,4 +1,28 @@
 <?xml version="1.0"?>
-<robot name="AGV_bot" xmlns:xacro="http://www.ros.org/wiki/xacro">
+<robot xmlns:xacro="http://www.ros.org/wiki/xacro" xmlns:gz="http://gazebosim.org/schema">
+    <xacro:macro name="wheel_collision" params="num">
+        <gazebo reference="wheel_link_${num}">
+            <collision>
+                <surface>
+                    <contact>
+                        <ode>
+                            <kp>1.5e6</kp>
+                            <kd>2e4</kd>
+                        </ode>
+                    </contact>
+                    <friction>
+                        <ode>
+                            <mu>0.6</mu>
+                            <mu2>0.1</mu2>
+                            <fdir1 gz:expressed_in="base_footprint">${-sin(num*pi*2/3)} ${cos(num*pi*2/3)} 0</fdir1>
+                        </ode>
+                    </friction>
+                </surface>
+            </collision>
+        </gazebo>
+    </xacro:macro>
+    <xacro:wheel_collision num="0" />
+    <xacro:wheel_collision num="1" />
+    <xacro:wheel_collision num="2" />
     <gazebo>
         <plugin filename="gz-sim-imu-system" name="gz::sim::systems::Imu">
